Commit message: Added and deleted config files. Added Town3 preplanned path config file and deleted obsolete files.

File: src/config/nuscenes.extrinsics.urdf (robot description, URDF)
Before this commit: robot example_robot, 13 links, 12 joints
Links:
- added link center
Joints:
- added joint base_link_to_center: type fixed, parent base_link, child center, origin xyz=1.4 0.0 -0.5 rpy=0.0 0.0 0.0
