Commit message: Changed post processing. Improved voxel visibility. Occupancy images are masked using voxel visibility masks (obstacles that are not visible in voxel space are masked out).

File: src/config/carla_extrinsics.urdf (robot description, URDF)
Before this commit: robot example_robot, 14 links, 13 joints
Joints:
- joint base_link_to_center: origin xyz=1.4 0.0 -0.5 rpy=0.0 0.0 0.0 -> xyz=0.8 0.0 0.5 rpy=0.0 0.0 0.0

Commit message: Converted simulation and postprocessing ipynb scripts to python scripts. Small adjustment in sensor spawning logic (urdf is parsed from base_link; center link is defined relative to base_link; all sensors are defined relative to center link)

File: src/config/carla_extrinsics.urdf (robot description, URDF)
Before this commit: robot example_robot, 14 links, 13 joints
Joints:
- joint base_link_to_CAM_BACK: parent base_link -> center
- joint base_link_to_CAM_BACK_LEFT: parent base_link -> center
- joint base_link_to_CAM_BACK_RIGHT: parent base_link -> center
- joint base_link_to_CAM_FRONT: parent base_link -> center
- joint base_link_to_CAM_FRONT_LEFT: parent base_link -> center
- joint base_link_to_CAM_FRONT_RIGHT: parent base_link -> center
- joint base_link_to_LIDAR_TOP: parent base_link -> center
- joint base_link_to_RADAR_BACK_LEFT: parent base_link -> center
- joint base_link_to_RADAR_BACK_RIGHT: parent base_link -> center
- joint base_link_to_RADAR_FRONT: parent base_link -> center
- joint base_link_to_RADAR_FRONT_LEFT: parent base_link -> center
- joint base_link_to_RADAR_FRONT_RIGHT: parent base_link -> center
- joint base_link_to_center: origin xyz=0.8 0.0 0.5 rpy=0.0 0.0 0.0 -> xyz=0.0 0.0 0.5 rpy=0.0 0.0 0.0

Commit message: Initial commit for recording simulation and performing separate sensor simulations based on the same recording.

File: src/config/carla_extrinsics.urdf (robot description, URDF)
Before this commit: robot example_robot, 14 links, 13 joints
Joints:
- joint base_link_to_center: origin xyz=0.0 0.0 0.5 rpy=0.0 0.0 0.0 -> xyz=-1.5 0.0 0.15 rpy=0.0 0.0 0.0
